Commit message: changed bone(head/tail)-position calculation, fixed the object-rotation issue

File: testing/urdf/r2d2.urdf (robot description, URDF)
Before this commit: robot visual, 16 links, 15 joints
Joints:
- joint base_to_right_leg: axis (none) -> 1 0 0; limit (none) -> lower=-0.5 upper=0.5 effort=40 velocity=10

Commit message: changed the bone-creation-algorithm, base_links visual will be created - if exist, also added the meka-urdf and changed the r2d2-joints to type=continuous for tests.

File: testing/urdf/r2d2.urdf (robot description, URDF)
Before this commit: robot visual, 16 links, 15 joints
Joints:
- joint base_to_left_leg: type fixed -> continuous
- joint base_to_right_leg: type fixed -> continuous
- joint gripper_extension: type fixed -> continuous
- joint head_swivel: type fixed -> continuous
- joint left_back_wheel_joint: type fixed -> continuous
- joint left_base_joint: type fixed -> continuous
- joint left_front_wheel_joint: type fixed -> continuous
- joint left_gripper_joint: type fixed -> continuous
- joint left_tip_joint: type fixed -> continuous
- joint right_back_wheel_joint: type fixed -> continuous
- joint right_base_joint: type fixed -> continuous
- joint right_front_wheel_joint: type fixed -> continuous
- joint right_gripper_joint: type fixed -> continuous
- joint right_tip_joint: type fixed -> continuous
- joint tobox: type fixed -> continuous

Commit message: changed/added joint configuration

File: testing/urdf/r2d2.urdf (robot description, URDF)
Before this commit: robot visual, 16 links, 15 joints
Joints:
- joint base_to_left_leg: type continuous -> revolute
- joint base_to_right_leg: type continuous -> revolute
- joint gripper_extension: type continuous -> revolute
- joint head_swivel: type continuous -> revolute
- joint left_back_wheel_joint: type continuous -> revolute
- joint left_base_joint: type continuous -> revolute
- joint left_front_wheel_joint: type continuous -> revolute
- joint left_gripper_joint: type continuous -> revolute
- joint left_tip_joint: type continuous -> revolute
- joint right_back_wheel_joint: type continuous -> revolute
- joint right_base_joint: type continuous -> revolute
- joint right_front_wheel_joint: type continuous -> revolute
- joint right_gripper_joint: type continuous -> revolute
- joint right_tip_joint: type continuous -> revolute
- joint tobox: type continuous -> revolute
