Commit message: let prismatic joints use the min-location limit, fixed issue with negative axis

File: testing/urdf/res/pepper.urdf (robot description, URDF)
Before this commit: robot JulietteY20MP, 84 links, 83 joints
Links:
- link Head: geometry collision mesh filename=res/pepper_meshes/meshes/1.0/HeadPitch_0.10.stl scale=1.0 1.0 1.0; visual mesh filename=res/pepper_meshes/meshes/1.0/HeadPitch.dae scale=1.0 1.0 1.0
- link Hip: geometry collision mesh filename=res/pepper_meshes/meshes/1.0/HipRoll_0.10.stl scale=1.0 1.0 1.0; visual mesh filename=res/pepper_meshes/meshes/1.0/HipRoll.dae scale=1.0 1.0 1.0
- link LBicep: geometry collision mesh filename=res/pepper_meshes/meshes/1.0/LShoulderRoll_0.10.stl scale=1.0 1.0 1.0; visual mesh filename=res/pepper_meshes/meshes/1.0/LShoulderRoll.dae scale=1.0 1.0 1.0
- link LElbow: geometry collision mesh filename=res/pepper_meshes/meshes/1.0/LElbowYaw_0.10.stl scale=1.0 1.0 1.0; visual mesh filename=res/pepper_meshes/meshes/1.0/LElbowYaw.dae scale=1.0 1.0 1.0
- link LFinger11_link: geometry collision mesh filename=res/pepper_meshes/meshes/1.0/LFinger11_0.10.stl scale=1.0 1.0 1.0; visual mesh filename=res/pepper_meshes/meshes/1.0/LFinger11.dae scale=1.0 1.0 1.0
- link LFinger12_link: geometry collision mesh filename=res/pepper_meshes/meshes/1.0/LFinger12_0.10.stl scale=1.0 1.0 1.0; visual mesh filename=res/pepper_meshes/meshes/1.0/LFinger12.dae scale=1.0 1.0 1.0
- link LFinger13_link: geometry collision mesh filename=res/pepper_meshes/meshes/1.0/LFinger13_0.10.stl scale=1.0 1.0 1.0; visual mesh filename=res/pepper_meshes/meshes/1.0/LFinger13.dae scale=1.0 1.0 1.0
- link LFinger21_link: geometry collision mesh filename=res/pepper_meshes/meshes/1.0/LFinger21_0.10.stl scale=1.0 1.0 1.0; visual mesh filename=res/pepper_meshes/meshes/1.0/LFinger21.dae scale=1.0 1.0 1.0
- link LFinger22_link: geometry collision mesh filename=res/pepper_meshes/meshes/1.0/LFinger22_0.10.stl scale=1.0 1.0 1.0; visual mesh filename=res/pepper_meshes/meshes/1.0/LFinger22.dae scale=1.0 1.0 1.0
- link LFinger23_link: geometry collision mesh filename=res/pepper_meshes/meshes/1.0/LFinger23_0.10.stl scale=1.0 1.0 1.0; visual mesh filename=res/pepper_meshes/meshes/1.0/LFinger23.dae scale=1.0 1.0 1.0
- link LFinger31_link: geometry collision mesh filename=res/pepper_meshes/meshes/1.0/LFinger31_0.10.stl scale=1.0 1.0 1.0; visual mesh filename=res/pepper_meshes/meshes/1.0/LFinger31.dae scale=1.0 1.0 1.0
- link LFinger32_link: geometry collision mesh filename=res/pepper_meshes/meshes/1.0/LFinger32_0.10.stl scale=1.0 1.0 1.0; visual mesh filename=res/pepper_meshes/meshes/1.0/LFinger32.dae scale=1.0 1.0 1.0
- link LFinger33_link: geometry collision mesh filename=res/pepper_meshes/meshes/1.0/LFinger33_0.10.stl scale=1.0 1.0 1.0; visual mesh filename=res/pepper_meshes/meshes/1.0/LFinger33.dae scale=1.0 1.0 1.0
- link LFinger41_link: geometry collision mesh filename=res/pepper_meshes/meshes/1.0/LFinger41_0.10.stl scale=1.0 1.0 1.0; visual mesh filename=res/pepper_meshes/meshes/1.0/LFinger41.dae scale=1.0 1.0 1.0
- link LFinger42_link: geometry collision mesh filename=res/pepper_meshes/meshes/1.0/LFinger42_0.10.stl scale=1.0 1.0 1.0; visual mesh filename=res/pepper_meshes/meshes/1.0/LFinger42.dae scale=1.0 1.0 1.0
- link LFinger43_link: geometry collision mesh filename=res/pepper_meshes/meshes/1.0/LFinger43_0.10.stl scale=1.0 1.0 1.0; visual mesh filename=res/pepper_meshes/meshes/1.0/LFinger43.dae scale=1.0 1.0 1.0
- link LForeArm: geometry collision mesh filename=res/pepper_meshes/meshes/1.0/LElbowRoll_0.10.stl scale=1.0 1.0 1.0; visual mesh filename=res/pepper_meshes/meshes/1.0/LElbowRoll.dae scale=1.0 1.0 1.0
- link LShoulder: geometry collision mesh filename=res/pepper_meshes/meshes/1.0/LShoulderPitch_0.10.stl scale=1.0 1.0 1.0; visual mesh filename=res/pepper_meshes/meshes/1.0/LShoulderPitch.dae scale=1.0 1.0 1.0
- link LThumb1_link: geometry collision mesh filename=res/pepper_meshes/meshes/1.0/LThumb1_0.10.stl scale=1.0 1.0 1.0; visual mesh filename=res/pepper_meshes/meshes/1.0/LThumb1.dae scale=1.0 1.0 1.0
- link LThumb2_link: geometry collision mesh filename=res/pepper_meshes/meshes/1.0/LThumb2_0.10.stl scale=1.0 1.0 1.0; visual mesh filename=res/pepper_meshes/meshes/1.0/LThumb2.dae scale=1.0 1.0 1.0
- link Neck: geometry collision mesh filename=res/pepper_meshes/meshes/1.0/HeadYaw_0.10.stl scale=1.0 1.0 1.0; visual mesh filename=res/pepper_meshes/meshes/1.0/HeadYaw.dae scale=1.0 1.0 1.0
- link Pelvis: geometry collision mesh filename=res/pepper_meshes/meshes/1.0/HipPitch_0.10.stl scale=1.0 1.0 1.0; visual mesh filename=res/pepper_meshes/meshes/1.0/HipPitch.dae scale=1.0 1.0 1.0
- link RBicep: geometry collision mesh filename=res/pepper_meshes/meshes/1.0/RShoulderRoll_0.10.stl scale=1.0 1.0 1.0; visual mesh filename=res/pepper_meshes/meshes/1.0/RShoulderRoll.dae scale=1.0 1.0 1.0
- link RElbow: geometry collision mesh filename=res/pepper_meshes/meshes/1.0/RElbowYaw_0.10.stl scale=1.0 1.0 1.0; visual mesh filename=res/pepper_meshes/meshes/1.0/RElbowYaw.dae scale=1.0 1.0 1.0
- link RFinger11_link: geometry collision mesh filename=res/pepper_meshes/meshes/1.0/RFinger11_0.10.stl scale=1.0 1.0 1.0; visual mesh filename=res/pepper_meshes/meshes/1.0/RFinger11.dae scale=1.0 1.0 1.0
- link RFinger12_link: geometry collision mesh filename=res/pepper_meshes/meshes/1.0/RFinger12_0.10.stl scale=1.0 1.0 1.0; visual mesh filename=res/pepper_meshes/meshes/1.0/RFinger12.dae scale=1.0 1.0 1.0
- link RFinger13_link: geometry collision mesh filename=res/pepper_meshes/meshes/1.0/RFinger13_0.10.stl scale=1.0 1.0 1.0; visual mesh filename=res/pepper_meshes/meshes/1.0/RFinger13.dae scale=1.0 1.0 1.0
- link RFinger21_link: geometry collision mesh filename=res/pepper_meshes/meshes/1.0/RFinger21_0.10.stl scale=1.0 1.0 1.0; visual mesh filename=res/pepper_meshes/meshes/1.0/RFinger21.dae scale=1.0 1.0 1.0
- link RFinger22_link: geometry collision mesh filename=res/pepper_meshes/meshes/1.0/RFinger22_0.10.stl scale=1.0 1.0 1.0; visual mesh filename=res/pepper_meshes/meshes/1.0/RFinger22.dae scale=1.0 1.0 1.0
- link RFinger23_link: geometry collision mesh filename=res/pepper_meshes/meshes/1.0/RFinger23_0.10.stl scale=1.0 1.0 1.0; visual mesh filename=res/pepper_meshes/meshes/1.0/RFinger23.dae scale=1.0 1.0 1.0
- link RFinger31_link: geometry collision mesh filename=res/pepper_meshes/meshes/1.0/RFinger31_0.10.stl scale=1.0 1.0 1.0; visual mesh filename=res/pepper_meshes/meshes/1.0/RFinger31.dae scale=1.0 1.0 1.0
- link RFinger32_link: geometry collision mesh filename=res/pepper_meshes/meshes/1.0/RFinger32_0.10.stl scale=1.0 1.0 1.0; visual mesh filename=res/pepper_meshes/meshes/1.0/RFinger32.dae scale=1.0 1.0 1.0
- link RFinger33_link: geometry collision mesh filename=res/pepper_meshes/meshes/1.0/RFinger33_0.10.stl scale=1.0 1.0 1.0; visual mesh filename=res/pepper_meshes/meshes/1.0/RFinger33.dae scale=1.0 1.0 1.0
- link RFinger41_link: geometry collision mesh filename=res/pepper_meshes/meshes/1.0/RFinger41_0.10.stl scale=1.0 1.0 1.0; visual mesh filename=res/pepper_meshes/meshes/1.0/RFinger41.dae scale=1.0 1.0 1.0
- link RFinger42_link: geometry collision mesh filename=res/pepper_meshes/meshes/1.0/RFinger42_0.10.stl scale=1.0 1.0 1.0; visual mesh filename=res/pepper_meshes/meshes/1.0/RFinger42.dae scale=1.0 1.0 1.0
- link RFinger43_link: geometry collision mesh filename=res/pepper_meshes/meshes/1.0/RFinger43_0.10.stl scale=1.0 1.0 1.0; visual mesh filename=res/pepper_meshes/meshes/1.0/RFinger43.dae scale=1.0 1.0 1.0
- link RForeArm: geometry collision mesh filename=res/pepper_meshes/meshes/1.0/RElbowRoll_0.10.stl scale=1.0 1.0 1.0; visual mesh filename=res/pepper_meshes/meshes/1.0/RElbowRoll.dae scale=1.0 1.0 1.0
- link RShoulder: geometry collision mesh filename=res/pepper_meshes/meshes/1.0/RShoulderPitch_0.10.stl scale=1.0 1.0 1.0; visual mesh filename=res/pepper_meshes/meshes/1.0/RShoulderPitch.dae scale=1.0 1.0 1.0
- link RThumb1_link: geometry collision mesh filename=res/pepper_meshes/meshes/1.0/RThumb1_0.10.stl scale=1.0 1.0 1.0; visual mesh filename=res/pepper_meshes/meshes/1.0/RThumb1.dae scale=1.0 1.0 1.0
- link RThumb2_link: geometry collision mesh filename=res/pepper_meshes/meshes/1.0/RThumb2_0.10.stl scale=1.0 1.0 1.0; visual mesh filename=res/pepper_meshes/meshes/1.0/RThumb2.dae scale=1.0 1.0 1.0
- link Tibia: geometry collision mesh filename=res/pepper_meshes/meshes/1.0/KneePitch_0.10.stl scale=1.0 1.0 1.0; visual mesh filename=res/pepper_meshes/meshes/1.0/KneePitch.dae scale=1.0 1.0 1.0
- link WheelB_link: geometry collision mesh filename=res/pepper_meshes/meshes/1.0/WheelB_0.10.stl scale=1.0 1.0 1.0; visual mesh filename=res/pepper_meshes/meshes/1.0/WheelB.dae scale=1.0 1.0 1.0
- link WheelFL_link: geometry collision mesh filename=res/pepper_meshes/meshes/1.0/WheelFL_0.10.stl scale=1.0 1.0 1.0; visual mesh filename=res/pepper_meshes/meshes/1.0/WheelFL.dae scale=1.0 1.0 1.0
- link WheelFR_link: geometry collision mesh filename=res/pepper_meshes/meshes/1.0/WheelFR_0.10.stl scale=1.0 1.0 1.0; visual mesh filename=res/pepper_meshes/meshes/1.0/WheelFR.dae scale=1.0 1.0 1.0
- link l_wrist: geometry collision mesh filename=res/pepper_meshes/meshes/1.0/LWristYaw_0.10.stl scale=1.0 1.0 1.0; visual mesh filename=res/pepper_meshes/meshes/1.0/LWristYaw.dae scale=1.0 1.0 1.0
- link r_wrist: geometry collision mesh filename=res/pepper_meshes/meshes/1.0/RWristYaw_0.10.stl scale=1.0 1.0 1.0; visual mesh filename=res/pepper_meshes/meshes/1.0/RWristYaw.dae scale=1.0 1.0 1.0
- link torso: geometry collision mesh filename=res/pepper_meshes/meshes/1.0/Torso_0.10.stl scale=1.0 1.0 1.0; visual mesh filename=res/pepper_meshes/meshes/1.0/Torso.dae scale=1.0 1.0 1.0

Commit message: changed the way the armature is built

File: testing/urdf/res/pepper.urdf (robot description, URDF)
Before this commit: robot JulietteY20MP, 84 links, 83 joints
Links:
- link Head: geometry collision mesh filename=res/pepper_meshes/meshes/1.0/HeadPitch_0.10.stl scale=0.3 0.3 0.3; visual mesh filename=res/pepper_meshes/meshes/1.0/HeadPitch.dae scale=0.3 0.3 0.3
- link Hip: geometry collision mesh filename=res/pepper_meshes/meshes/1.0/HipRoll_0.10.stl scale=0.3 0.3 0.3; visual mesh filename=res/pepper_meshes/meshes/1.0/HipRoll.dae scale=0.3 0.3 0.3
- link LBicep: geometry collision mesh filename=res/pepper_meshes/meshes/1.0/LShoulderRoll_0.10.stl scale=0.3 0.3 0.3; visual mesh filename=res/pepper_meshes/meshes/1.0/LShoulderRoll.dae scale=0.3 0.3 0.3
- link LElbow: geometry collision mesh filename=res/pepper_meshes/meshes/1.0/LElbowYaw_0.10.stl scale=0.3 0.3 0.3; visual mesh filename=res/pepper_meshes/meshes/1.0/LElbowYaw.dae scale=0.3 0.3 0.3
- link LFinger11_link: geometry collision mesh filename=res/pepper_meshes/meshes/1.0/LFinger11_0.10.stl scale=0.3 0.3 0.3; visual mesh filename=res/pepper_meshes/meshes/1.0/LFinger11.dae scale=0.3 0.3 0.3
- link LFinger12_link: geometry collision mesh filename=res/pepper_meshes/meshes/1.0/LFinger12_0.10.stl scale=0.3 0.3 0.3; visual mesh filename=res/pepper_meshes/meshes/1.0/LFinger12.dae scale=0.3 0.3 0.3
- link LFinger13_link: geometry collision mesh filename=res/pepper_meshes/meshes/1.0/LFinger13_0.10.stl scale=0.3 0.3 0.3; visual mesh filename=res/pepper_meshes/meshes/1.0/LFinger13.dae scale=0.3 0.3 0.3
- link LFinger21_link: geometry collision mesh filename=res/pepper_meshes/meshes/1.0/LFinger21_0.10.stl scale=0.3 0.3 0.3; visual mesh filename=res/pepper_meshes/meshes/1.0/LFinger21.dae scale=0.3 0.3 0.3
- link LFinger22_link: geometry collision mesh filename=res/pepper_meshes/meshes/1.0/LFinger22_0.10.stl scale=0.3 0.3 0.3; visual mesh filename=res/pepper_meshes/meshes/1.0/LFinger22.dae scale=0.3 0.3 0.3
- link LFinger23_link: geometry collision mesh filename=res/pepper_meshes/meshes/1.0/LFinger23_0.10.stl scale=0.3 0.3 0.3; visual mesh filename=res/pepper_meshes/meshes/1.0/LFinger23.dae scale=0.3 0.3 0.3
- link LFinger31_link: geometry collision mesh filename=res/pepper_meshes/meshes/1.0/LFinger31_0.10.stl scale=0.3 0.3 0.3; visual mesh filename=res/pepper_meshes/meshes/1.0/LFinger31.dae scale=0.3 0.3 0.3
- link LFinger32_link: geometry collision mesh filename=res/pepper_meshes/meshes/1.0/LFinger32_0.10.stl scale=0.3 0.3 0.3; visual mesh filename=res/pepper_meshes/meshes/1.0/LFinger32.dae scale=0.3 0.3 0.3
- link LFinger33_link: geometry collision mesh filename=res/pepper_meshes/meshes/1.0/LFinger33_0.10.stl scale=0.3 0.3 0.3; visual mesh filename=res/pepper_meshes/meshes/1.0/LFinger33.dae scale=0.3 0.3 0.3
- link LFinger41_link: geometry collision mesh filename=res/pepper_meshes/meshes/1.0/LFinger41_0.10.stl scale=0.3 0.3 0.3; visual mesh filename=res/pepper_meshes/meshes/1.0/LFinger41.dae scale=0.3 0.3 0.3
- link LFinger42_link: geometry collision mesh filename=res/pepper_meshes/meshes/1.0/LFinger42_0.10.stl scale=0.3 0.3 0.3; visual mesh filename=res/pepper_meshes/meshes/1.0/LFinger42.dae scale=0.3 0.3 0.3
- link LFinger43_link: geometry collision mesh filename=res/pepper_meshes/meshes/1.0/LFinger43_0.10.stl scale=0.3 0.3 0.3; visual mesh filename=res/pepper_meshes/meshes/1.0/LFinger43.dae scale=0.3 0.3 0.3
- link LForeArm: geometry collision mesh filename=res/pepper_meshes/meshes/1.0/LElbowRoll_0.10.stl scale=0.3 0.3 0.3; visual mesh filename=res/pepper_meshes/meshes/1.0/LElbowRoll.dae scale=0.3 0.3 0.3
- link LShoulder: geometry collision mesh filename=res/pepper_meshes/meshes/1.0/LShoulderPitch_0.10.stl scale=0.3 0.3 0.3; visual mesh filename=res/pepper_meshes/meshes/1.0/LShoulderPitch.dae scale=0.3 0.3 0.3
- link LThumb1_link: geometry collision mesh filename=res/pepper_meshes/meshes/1.0/LThumb1_0.10.stl scale=0.3 0.3 0.3; visual mesh filename=res/pepper_meshes/meshes/1.0/LThumb1.dae scale=0.3 0.3 0.3
- link LThumb2_link: geometry collision mesh filename=res/pepper_meshes/meshes/1.0/LThumb2_0.10.stl scale=0.3 0.3 0.3; visual mesh filename=res/pepper_meshes/meshes/1.0/LThumb2.dae scale=0.3 0.3 0.3
- link Neck: geometry collision mesh filename=res/pepper_meshes/meshes/1.0/HeadYaw_0.10.stl scale=0.3 0.3 0.3; visual mesh filename=res/pepper_meshes/meshes/1.0/HeadYaw.dae scale=0.3 0.3 0.3
- link Pelvis: geometry collision mesh filename=res/pepper_meshes/meshes/1.0/HipPitch_0.10.stl scale=0.3 0.3 0.3; visual mesh filename=res/pepper_meshes/meshes/1.0/HipPitch.dae scale=0.3 0.3 0.3
- link RBicep: geometry collision mesh filename=res/pepper_meshes/meshes/1.0/RShoulderRoll_0.10.stl scale=0.3 0.3 0.3; visual mesh filename=res/pepper_meshes/meshes/1.0/RShoulderRoll.dae scale=0.3 0.3 0.3
- link RElbow: geometry collision mesh filename=res/pepper_meshes/meshes/1.0/RElbowYaw_0.10.stl scale=0.3 0.3 0.3; visual mesh filename=res/pepper_meshes/meshes/1.0/RElbowYaw.dae scale=0.3 0.3 0.3
- link RFinger11_link: geometry collision mesh filename=res/pepper_meshes/meshes/1.0/RFinger11_0.10.stl scale=0.3 0.3 0.3; visual mesh filename=res/pepper_meshes/meshes/1.0/RFinger11.dae scale=0.3 0.3 0.3
- link RFinger12_link: geometry collision mesh filename=res/pepper_meshes/meshes/1.0/RFinger12_0.10.stl scale=0.3 0.3 0.3; visual mesh filename=res/pepper_meshes/meshes/1.0/RFinger12.dae scale=0.3 0.3 0.3
- link RFinger13_link: geometry collision mesh filename=res/pepper_meshes/meshes/1.0/RFinger13_0.10.stl scale=0.3 0.3 0.3; visual mesh filename=res/pepper_meshes/meshes/1.0/RFinger13.dae scale=0.3 0.3 0.3
- link RFinger21_link: geometry collision mesh filename=res/pepper_meshes/meshes/1.0/RFinger21_0.10.stl scale=0.3 0.3 0.3; visual mesh filename=res/pepper_meshes/meshes/1.0/RFinger21.dae scale=0.3 0.3 0.3
- link RFinger22_link: geometry collision mesh filename=res/pepper_meshes/meshes/1.0/RFinger22_0.10.stl scale=0.3 0.3 0.3; visual mesh filename=res/pepper_meshes/meshes/1.0/RFinger22.dae scale=0.3 0.3 0.3
- link RFinger23_link: geometry collision mesh filename=res/pepper_meshes/meshes/1.0/RFinger23_0.10.stl scale=0.3 0.3 0.3; visual mesh filename=res/pepper_meshes/meshes/1.0/RFinger23.dae scale=0.3 0.3 0.3
- link RFinger31_link: geometry collision mesh filename=res/pepper_meshes/meshes/1.0/RFinger31_0.10.stl scale=0.3 0.3 0.3; visual mesh filename=res/pepper_meshes/meshes/1.0/RFinger31.dae scale=0.3 0.3 0.3
- link RFinger32_link: geometry collision mesh filename=res/pepper_meshes/meshes/1.0/RFinger32_0.10.stl scale=0.3 0.3 0.3; visual mesh filename=res/pepper_meshes/meshes/1.0/RFinger32.dae scale=0.3 0.3 0.3
- link RFinger33_link: geometry collision mesh filename=res/pepper_meshes/meshes/1.0/RFinger33_0.10.stl scale=0.3 0.3 0.3; visual mesh filename=res/pepper_meshes/meshes/1.0/RFinger33.dae scale=0.3 0.3 0.3
- link RFinger41_link: geometry collision mesh filename=res/pepper_meshes/meshes/1.0/RFinger41_0.10.stl scale=0.3 0.3 0.3; visual mesh filename=res/pepper_meshes/meshes/1.0/RFinger41.dae scale=0.3 0.3 0.3
- link RFinger42_link: geometry collision mesh filename=res/pepper_meshes/meshes/1.0/RFinger42_0.10.stl scale=0.3 0.3 0.3; visual mesh filename=res/pepper_meshes/meshes/1.0/RFinger42.dae scale=0.3 0.3 0.3
- link RFinger43_link: geometry collision mesh filename=res/pepper_meshes/meshes/1.0/RFinger43_0.10.stl scale=0.3 0.3 0.3; visual mesh filename=res/pepper_meshes/meshes/1.0/RFinger43.dae scale=0.3 0.3 0.3
- link RForeArm: geometry collision mesh filename=res/pepper_meshes/meshes/1.0/RElbowRoll_0.10.stl scale=0.3 0.3 0.3; visual mesh filename=res/pepper_meshes/meshes/1.0/RElbowRoll.dae scale=0.3 0.3 0.3
- link RShoulder: geometry collision mesh filename=res/pepper_meshes/meshes/1.0/RShoulderPitch_0.10.stl scale=0.3 0.3 0.3; visual mesh filename=res/pepper_meshes/meshes/1.0/RShoulderPitch.dae scale=0.3 0.3 0.3
- link RThumb1_link: geometry collision mesh filename=res/pepper_meshes/meshes/1.0/RThumb1_0.10.stl scale=0.3 0.3 0.3; visual mesh filename=res/pepper_meshes/meshes/1.0/RThumb1.dae scale=0.3 0.3 0.3
- link RThumb2_link: geometry collision mesh filename=res/pepper_meshes/meshes/1.0/RThumb2_0.10.stl scale=0.3 0.3 0.3; visual mesh filename=res/pepper_meshes/meshes/1.0/RThumb2.dae scale=0.3 0.3 0.3
- link Tibia: geometry collision mesh filename=res/pepper_meshes/meshes/1.0/KneePitch_0.10.stl scale=0.3 0.3 0.3; visual mesh filename=res/pepper_meshes/meshes/1.0/KneePitch.dae scale=0.3 0.3 0.3
- link WheelB_link: geometry collision mesh filename=res/pepper_meshes/meshes/1.0/WheelB_0.10.stl scale=0.3 0.3 0.3; visual mesh filename=res/pepper_meshes/meshes/1.0/WheelB.dae scale=0.3 0.3 0.3
- link WheelFL_link: geometry collision mesh filename=res/pepper_meshes/meshes/1.0/WheelFL_0.10.stl scale=0.3 0.3 0.3; visual mesh filename=res/pepper_meshes/meshes/1.0/WheelFL.dae scale=0.3 0.3 0.3
- link WheelFR_link: geometry collision mesh filename=res/pepper_meshes/meshes/1.0/WheelFR_0.10.stl scale=0.3 0.3 0.3; visual mesh filename=res/pepper_meshes/meshes/1.0/WheelFR.dae scale=0.3 0.3 0.3
- link l_wrist: geometry collision mesh filename=res/pepper_meshes/meshes/1.0/LWristYaw_0.10.stl scale=0.3 0.3 0.3; visual mesh filename=res/pepper_meshes/meshes/1.0/LWristYaw.dae scale=0.3 0.3 0.3
- link r_wrist: geometry collision mesh filename=res/pepper_meshes/meshes/1.0/RWristYaw_0.10.stl scale=0.3 0.3 0.3; visual mesh filename=res/pepper_meshes/meshes/1.0/RWristYaw.dae scale=0.3 0.3 0.3
- link torso: geometry collision mesh filename=res/pepper_meshes/meshes/1.0/Torso_0.10.stl scale=0.3 0.3 0.3; visual mesh filename=res/pepper_meshes/meshes/1.0/Torso.dae scale=0.3 0.3 0.3
