Commit message: recoded the built of armature

File: testing/urdf/res/r2d2.urdf (robot description, URDF)
Before this commit: robot visual, 16 links, 15 joints
Links:
- link left_gripper: geometry visual mesh filename=package://urdf_tutorial/meshes/l_finger.dae
- link left_tip: geometry visual mesh filename=package://urdf_tutorial/meshes/l_finger_tip.dae
- link right_gripper: geometry visual mesh filename=package://urdf_tutorial/meshes/l_finger.dae
- link right_tip: geometry visual mesh filename=package://urdf_tutorial/meshes/l_finger_tip.dae
Joints:
- joint base_to_left_leg: type revolute -> fixed
- joint base_to_right_leg: axis 1 0 0 -> (none); limit lower=-0.5 upper=0.5 effort=40 velocity=10 -> (none); type revolute -> fixed
- joint gripper_extension: type revolute -> fixed
- joint head_swivel: type revolute -> fixed
- joint left_back_wheel_joint: type revolute -> fixed
- joint left_base_joint: type revolute -> fixed
- joint left_front_wheel_joint: type revolute -> fixed
- joint left_gripper_joint: type revolute -> fixed
- joint left_tip_joint: type revolute -> fixed
- joint right_back_wheel_joint: type revolute -> fixed
- joint right_base_joint: type revolute -> fixed
- joint right_front_wheel_joint: type revolute -> fixed
- joint right_gripper_joint: type revolute -> fixed
- joint right_tip_joint: type revolute -> fixed
- joint tobox: type revolute -> fixed
